Commit message: urdf

File: code/src/husky_description/urdf/decorations.urdf.xacro (robot description, xacro)
@@ -97,6 +97,7 @@
       </joint>
     </xacro:if>
-    <xacro:if value="$(optenv HUSKY_TOP_PLATE_ENABLED true)">
-      <!-- Spawn the top plate -->
+  <!-- COMMENTED OUT - ØØ 21.02.2023
+    <xacro:if value="$(optenv HUSKY_TOP_PLATE_ENABLED true)">-->
+      <!-- Spawn the top plate
       <xacro:if value="$(optenv HUSKY_LARGE_TOP_PLATE false)">
         <link name="top_plate_link">
@@ -113,18 +114,18 @@
             </geometry>
           </collision>
-        </link>
-        <!-- Attach top plate -->
+        </link>-->
+        <!-- Attach top plate
         <joint name="top_plate_joint" type="fixed">
           <parent link="base_link" />
           <child link="top_plate_link"/>
           <origin xyz="0.0812 0 0.225" rpy="0 0 0"/>
-        </joint>
-        <!-- Top plate front link -->
+        </joint>-->
+        <!-- Top plate front link
         <joint name="top_plate_front_joint" type="fixed">
           <parent link="top_plate_link" />
           <child link="top_plate_front_link"/>
           <origin xyz="0.4125 0 0.00672" rpy="0 0 0"/>
-        </joint>
-        <!-- Top plate rear link-->
+        </joint>-->
+        <!-- Top plate rear link
         <joint name="top_plate_rear_joint" type="fixed">
           <parent link="top_plate_link" />
@@ -147,18 +148,18 @@
             </geometry>
           </collision>
-        </link>
-        <!-- Attach top plate -->
+        </link>-->
+        <!-- Attach top plate
         <joint name="top_plate_joint" type="fixed">
           <parent link="base_link" />
           <child link="top_plate_link"/>
           <origin xyz="0.0812 0 0.245" rpy="0 0 0"/>
-        </joint>
-        <!-- Top plate front link -->
+        </joint>-->
+        <!-- Top plate front link
         <joint name="top_plate_front_joint" type="fixed">
           <parent link="top_plate_link" />
           <child link="top_plate_front_link"/>
           <origin xyz="0.36367 0 0.00639" rpy="0 0 0"/>
-        </joint>
-        <!-- Top plate rear link-->
+        </joint>-->
+        <!-- Top plate rear link
         <joint name="top_plate_rear_joint" type="fixed">
           <parent link="top_plate_link" />
@@ -170,4 +171,5 @@
       <link name="top_plate_rear_link"/>
     </xacro:if>
+   -->
   </xacro:macro>
 </robot>
