Commit message: added frame to urdf

File: code/src/husky_description/urdf/husky.urdf.xacro (robot description, xacro)
@@ -43,5 +43,50 @@
   <!-- Optional custom includes. -->
   <!-- THIS IS COMMENTED OUT BY ØØ, HUSKY PROJECT <xacro:include filename="$(arg urdf_extras)" /> -->
-  <!-- OUSTER LIDAR LINK. ØØ. 19.09.22 -->
+  <link
+    name="frame_link">
+    <inertial>
+      <origin
+        xyz="-0.019514 -0.052513 0.024073"
+        rpy="0 0 0" />
+      <mass
+        value="1.5326" />
+      <inertia
+        ixx="0.025107"
+        ixy="7.1994E-19"
+        ixz="-4.8558E-21"
+        iyy="0.004688"
+        iyz="9.2216E-19"
+        izz="0.020746" />
+    </inertial>
+    <visual>
+      <origin
+        xyz="0 0 0"
+        rpy="0 0 0" />
+      <geometry>
+        <mesh
+          filename="file://$(find husky_description)/meshes/frame_link.STL" />
+      </geometry>
+      <material
+        name="">
+        <color
+          rgba="0.89804 0.91765 0.92941 1" />
+      </material>
+    </visual>
+    <collision>
+      <origin
+        xyz="0 0 0"
+        rpy="0 0 0" />
+      <geometry>
+        <mesh
+          filename="file://$(find husky_description)/meshes/frame_link.STL" />
+      </geometry>
+    </collision>
+  </link>
+  <joint name="frame_joint" type="fixed">
+    <parent link="user_rail_link"/>
+    <child link="frame_link"/>
+    <origin xyz="0 0 0.3" rpy="-1.57079633 0 0"/>
+  </joint>
+  <!-- OUSTER LIDAR LINK. ØØ. 19.09.22
   <link name="lidar_link">
     <inertial>
@@ -63,10 +108,10 @@
     </visual>
   </link>
-  <joint name="lidar_join" type="fixed">
+  <joint name="lidar_joint" type="fixed">
     <parent link="base_link"/>
     <child link="lidar_link"/>
     <origin xyz="0.175 0 0.505" rpy="0 0 3.14"/>
-  </joint>
-  <!-- OUSTER LIDAR GAZEBO. ØØ. 19.09.22 -->
+  </joint> -->
+  <!-- OUSTER LIDAR GAZEBO. ØØ. 19.09.22
   <gazebo reference="lidar_link">
     <sensor name="lidar" type="ray">
@@ -103,3 +148,4 @@
     </sensor>
   </gazebo>
+  -->
 </robot>

Commit message: EUREKA! URDF

File: code/src/husky_description/urdf/husky.urdf.xacro (robot description, xacro)
@@ -47,15 +47,15 @@
     <inertial>
       <origin
-        xyz="-0.019514 -0.052513 0.024073"
+        xyz="0 0 0"
         rpy="0 0 0" />
       <mass
-        value="1.5326" />
+        value="2.2936" />
       <inertia
-        ixx="0.025107"
-        ixy="7.1994E-19"
-        ixz="-4.8558E-21"
-        iyy="0.004688"
-        iyz="9.2216E-19"
-        izz="0.020746" />
+        ixx="0.026381"
+        ixy="1.2862E-08"
+        ixz="-2.2196E-07"
+        iyy="0.021942"
+        iyz="2.0183E-08"
+        izz="0.0063606" />
     </inertial>
     <visual>
@@ -86,5 +86,5 @@
     <parent link="user_rail_link"/>
     <child link="frame_link"/>
-    <origin xyz="0 0 0.3" rpy="-1.57079633 0 0"/>
+    <origin xyz="-0.01 0 0.01" rpy="0 0 0"/>
   </joint>
   <!-- OUSTER LIDAR LINK. ØØ. 19.09.22
