Commit message: genious

File: code/src/husky_group/urdf/husky_urdf_extras.urdf (robot description, URDF)
Before this commit: robot None, 2 links, 2 joints
Links:
- removed link lidar_link
Joints:
- joint lidar_joint: origin xyz=-0.0635 0 0.610 rpy=0 0 3.14 -> xyz=-0.0635 0 0.610 rpy=0 0 0

Commit message: fix

File: code/src/husky_group/urdf/husky_urdf_extras.urdf (robot description, URDF)
Before this commit: robot None, 1 links, 2 joints
Links:
- added link lidar_link

Commit message: flipped lidar

File: code/src/husky_group/urdf/husky_urdf_extras.urdf (robot description, URDF)
Before this commit: robot None, 2 links, 2 joints
Joints:
- joint lidar_joint: origin xyz=-0.0635 0 0.610 rpy=0 0 0 -> xyz=-0.0635 0 0.610 rpy=0 0 3.14

Commit message: flipped lidar back

File: code/src/husky_group/urdf/husky_urdf_extras.urdf (robot description, URDF)
Before this commit: robot None, 2 links, 2 joints
Joints:
- joint lidar_joint: origin xyz=-0.0635 0 0.610 rpy=0 0 3.14 -> xyz=-0.0635 0 0.610 rpy=0 0 0

Commit message: added realsense link to urdf

File: code/src/husky_group/urdf/husky_urdf_extras.urdf (robot description, URDF)
Before this commit: robot None, 2 links, 2 joints
Links:
- added link camera_link
Joints:
- added joint realsense_joint: type fixed, parent vx300/ee_gripper_link, child camera_link, origin xyz=0 0 0.05 rpy=0 0 0

Commit message: added black to lidar

File: code/src/husky_group/urdf/husky_urdf_extras.urdf (robot description, URDF)
Before this commit: robot None, 2 links, 2 joints
Links:
- link lidar_link: geometry visual cylinder length=0.03 radius=0.039

Commit message: [husky_group] change to package path

File: code/src/husky_group/urdf/husky_urdf_extras.urdf (robot description, URDF)
Before this commit: robot None, 2 links, 2 joints
Links:
- link frame_link: geometry collision mesh filename=package://husky_group/meshes/frame_link.STL; visual mesh filename=package://husky_group/meshes/frame_link.STL

Commit message: added realsense camera

File: code/src/husky_group/urdf/husky_urdf_extras.urdf (robot description, URDF)
Before this commit: robot None, 2 links, 2 joints
Links:
- added link camera_link; collision mesh filename=package://husky_group/meshes/realsense_assembly.STL; visual mesh filename=package://husky_group/meshes/realsense_assembly.STL

Commit message: urdf test

File: code/src/husky_group/urdf/husky_urdf_extras.urdf (robot description, URDF)
Before this commit: robot None, 3 links, 2 joints
Joints:
- added joint camera_joint: type fixed, parent vx300/ee_gripper_link, child camera_link, origin xyz=0 0 0.05 rpy=0 0 0

Commit message: does this work?

File: code/src/husky_group/urdf/husky_urdf_extras.urdf (robot description, URDF)
Before this commit: robot None, 3 links, 3 joints
Links:
- added link vx300/ee_gripper_link

Commit message: does this work then?

File: code/src/husky_group/urdf/husky_urdf_extras.urdf (robot description, URDF)
Before this commit: robot None, 4 links, 3 joints
Links:
- removed link vx300/ee_gripper_link
Joints:
- removed joint camera_joint

Commit message: see if it is the mesh

File: code/src/husky_group/urdf/husky_urdf_extras.urdf (robot description, URDF)
Before this commit: robot None, 3 links, 2 joints
Links:
- link camera_link: geometry collision cylinder length=0.03 radius=0.039; visual cylinder length=0.03 radius=0.039
