Commit message: safd

File: code/src/husky_group/urdf/interbotix_urdf_extras.urdf (robot description, URDF)
Before this commit: robot None, 1 links, 1 joints
Links:
- link camera_link: geometry collision mesh filename=package://husky_group/meshes/realsense_assembly.STL; visual mesh filename=package://husky_group/meshes/realsense_assembly.STL

Commit message: typo

File: code/src/husky_group/urdf/interbotix_urdf_extras.urdf (robot description, URDF)
Before this commit: robot None, 1 links, 1 joints
Links:
- link camera_link: geometry collision mesh filename=package://husky_group/meshes/Realsense_assembly.STL; visual mesh filename=package://husky_group/meshes/Realsense_assembly.STL

Commit message: testing

File: code/src/husky_group/urdf/interbotix_urdf_extras.urdf (robot description, URDF)
Before this commit: robot None, 1 links, 1 joints
Links:
- link camera_link: mass None -> 0.064463; geometry collision mesh filename=package://husky_group/meshes/camera_link.STL; visual mesh filename=package://husky_group/meshes/camera_link.STL

Commit message: hmmm

File: code/src/husky_group/urdf/interbotix_urdf_extras.urdf (robot description, URDF)
Before this commit: robot None, 1 links, 1 joints
Links:
- link camera_link: geometry collision cylinder length=0.03 radius=0.039; visual mesh filename=package://husky_group/meshes/camera_link.STL

Commit message: change to small letters

File: code/src/husky_group/urdf/interbotix_urdf_extras.urdf (robot description, URDF)
Before this commit: robot None, 1 links, 1 joints
Links:
- link camera_link: geometry collision cylinder length=0.03 radius=0.039; visual mesh filename=package://husky_group/meshes/camera_link.stl

Commit message: some work

File: code/src/husky_group/urdf/interbotix_urdf_extras.urdf (robot description, URDF)
Before this commit: robot None, 1 links, 1 joints
Links:
- link camera_link: geometry collision mesh filename=package://husky_group/meshes/camera_link.stl; visual mesh filename=package://husky_group/meshes/camera_link.STL
Joints:
- joint realsense_joint: origin xyz=0 0 0.1 rpy=0 0 0 -> xyz=0.028 0 0.035 rpy=0 0 0
