Commit message: inplementing cam

File: code/src/husky_interbotix/urdf/interbotix_urdf_extras.urdf (robot description, URDF)
Before this commit: robot None, 1 links, 1 joints
Links:
- added link camera_frame_link, mass 0.064463; collision mesh filename=package://husky_interbotix/meshes/camera_link.stl; visual mesh filename=package://husky_interbotix/meshes/camera_link.STL
- link camera_link: mass 0.064463 -> None; geometry 
Joints:
- added joint camera_frame_joint: type fixed, parent $(arg robot_name)/gripper_link, child camera_frame_link, origin xyz=0.028 0 0.035 rpy=0 0 0
- joint realsense_joint: origin xyz=0.028 0 0.035 rpy=0 0 0 -> xyz=0.03 0 0.03 rpy=0 ${pi/2} -${pi/2}; parent $(arg robot_name)/gripper_link -> camera_frame_link

Commit message: [husky_interbotix] urdf fix

File: code/src/husky_interbotix/urdf/interbotix_urdf_extras.urdf (robot description, URDF)
Before this commit: robot None, 2 links, 2 joints
Joints:
- joint realsense_joint: origin xyz=0.03 0 0.03 rpy=0 ${pi/2} -${pi/2} -> xyz=0.03 0 0.035 rpy=0 0 0

Commit message: [husky_interbotix] camera orientation

File: code/src/husky_interbotix/urdf/interbotix_urdf_extras.urdf (robot description, URDF)
Before this commit: robot None, 2 links, 2 joints
Joints:
- joint realsense_joint: origin xyz=0.03 0 0.035 rpy=0 0 0 -> xyz=0.03 0 0.035 rpy=0 ${pi/2} 0

Commit message: [husky_interbotix] camera_link orientation

File: code/src/husky_interbotix/urdf/interbotix_urdf_extras.urdf (robot description, URDF)
Before this commit: robot None, 2 links, 2 joints
Joints:
- joint realsense_joint: origin xyz=0.03 0 0.035 rpy=0 ${pi/2} 0 -> xyz=0.03 0 0.035 rpy=0 ${pi/2} ${pi}

Commit message: [husky_interbotix] cam_link orientation

File: code/src/husky_interbotix/urdf/interbotix_urdf_extras.urdf (robot description, URDF)
Before this commit: robot None, 2 links, 2 joints
Joints:
- joint realsense_joint: origin xyz=0.03 0 0.035 rpy=0 ${pi/2} ${pi} -> xyz=0.03 0 0.035 rpy=0 -${pi/2} ${pi}

Commit message: [husky_interbotix] camera_link orientation

File: code/src/husky_interbotix/urdf/interbotix_urdf_extras.urdf (robot description, URDF)
Before this commit: robot None, 2 links, 2 joints
Joints:
- joint realsense_joint: origin xyz=0.03 0 0.035 rpy=0 -${pi/2} ${pi} -> xyz=0.025 0 0.035 rpy=0 -${pi/2} ${pi/2}

Commit message: [husky_interbotix] camera_link makes no sense

File: code/src/husky_interbotix/urdf/interbotix_urdf_extras.urdf (robot description, URDF)
Before this commit: robot None, 2 links, 2 joints
Joints:
- joint realsense_joint: origin xyz=0.025 0 0.035 rpy=0 -${pi/2} ${pi/2} -> xyz=0.025 0 0.035 rpy=0 ${pi/2} 0

Commit message: [husky_interbotix] pitch pi, yaw pi

File: code/src/husky_interbotix/urdf/interbotix_urdf_extras.urdf (robot description, URDF)
Before this commit: robot None, 2 links, 2 joints
Joints:
- joint realsense_joint: origin xyz=0.025 0 0.035 rpy=0 ${pi/2} 0 -> xyz=0.025 0 0.035 rpy=0 ${pi} ${pi}

Commit message: [husky_interbotix] camera_link

File: code/src/husky_interbotix/urdf/interbotix_urdf_extras.urdf (robot description, URDF)
Before this commit: robot None, 2 links, 2 joints
Joints:
- joint realsense_joint: origin xyz=0.025 0 0.035 rpy=0 ${pi} ${pi} -> xyz=0.025 0 0.035 rpy=${pi/2} 0 ${pi/2}

Commit message: [husky_interbotix]  move camera link

File: code/src/husky_interbotix/urdf/interbotix_urdf_extras.urdf (robot description, URDF)
Before this commit: robot None, 2 links, 2 joints
Joints:
- joint realsense_joint: origin xyz=0.025 0 0.035 rpy=${pi/2} 0 ${pi/2} -> xyz=0.035 0 0.025 rpy=${pi/2} 0 ${pi/2}

Commit message: [husky_interbotix] camera_link orientation

File: code/src/husky_interbotix/urdf/interbotix_urdf_extras.urdf (robot description, URDF)
Before this commit: robot None, 2 links, 2 joints
Joints:
- joint realsense_joint: origin xyz=0.035 0 0.025 rpy=${pi/2} 0 ${pi/2} -> xyz=0.035 0 0.025 rpy=-${pi/2} 0 ${pi/2}

Commit message: camera orientatiuo n

File: code/src/husky_interbotix/urdf/interbotix_urdf_extras.urdf (robot description, URDF)
Before this commit: robot None, 2 links, 2 joints
Joints:
- joint realsense_joint: origin xyz=0.035 0 0.025 rpy=-${pi/2} 0 ${pi/2} -> xyz=0.035 0 0.025 rpy=-${pi/2} 0 -${pi/2}

Commit message: [interbotix_husky] realsense camera urdf shit

File: code/src/husky_interbotix/urdf/interbotix_urdf_extras.urdf (robot description, URDF)
Before this commit: robot None, 2 links, 2 joints
Joints:
- joint realsense_joint: origin xyz=0.035 0 0.025 rpy=-${pi/2} 0 -${pi/2} -> xyz=0.035 0 0.025 rpy=0 0 0

Commit message: cmon man

File: code/src/husky_interbotix/urdf/interbotix_urdf_extras.urdf (robot description, URDF)
Before this commit: robot None, 2 links, 2 joints
Links:
- added link $(arg robot_name)/ee_link
Joints:
- joint realsense_joint: child camera_link -> (arg robot_name)/ee_link; origin xyz=0.035 0 0.025 rpy=0 0 0 -> xyz=0 0 0 rpy=0 -${pi/2} 0; parent camera_frame_link -> $(arg robot_name)/ee_gripper_link

Commit message: fix

File: code/src/husky_interbotix/urdf/interbotix_urdf_extras.urdf (robot description, URDF)
Before this commit: robot None, 3 links, 2 joints
Joints:
- joint realsense_joint: child (arg robot_name)/ee_link -> $(arg robot_name)/ee_link

Commit message: woops

File: code/src/husky_interbotix/urdf/interbotix_urdf_extras.urdf (robot description, URDF)
Before this commit: robot None, 3 links, 2 joints
Joints:
- added joint ee_joint: type fixed, parent $(arg robot_name)/ee_gripper_link, child $(arg robot_name)/ee_link, origin xyz=0 0 0 rpy=0 -${pi/2} 0
- joint realsense_joint: child $(arg robot_name)/ee_link -> camera_link; origin xyz=0 0 0 rpy=0 -${pi/2} 0 -> xyz=0.035 0 0.025 rpy=0 0 0; parent $(arg robot_name)/ee_gripper_link -> camera_frame_link

Commit message: fask

File: code/src/husky_interbotix/urdf/interbotix_urdf_extras.urdf (robot description, URDF)
Before this commit: robot None, 5 links, 5 joints
Links:
- link camera_frame_link: geometry collision mesh filename=package://husky_interbotix/meshes/camera_link.STL; visual mesh filename=package://husky_interbotix/meshes/camera_link.STL

Commit message: commit changes

File: code/src/husky_interbotix/urdf/interbotix_urdf_extras.urdf (robot description, URDF)
Before this commit: robot None, 5 links, 5 joints
Links:
- removed link $(arg robot_name)/ee_gripper_link
- removed link $(arg robot_name)/left_finger_link
- removed link $(arg robot_name)/right_finger_link
Joints:
- removed joint ee_gripper
- removed joint left_finger
- removed joint right_finger

Commit message: just a testjust a test

File: code/src/husky_interbotix/urdf/interbotix_urdf_extras.urdf (robot description, URDF)
Before this commit: robot None, 2 links, 2 joints
Links:
- added link $(arg robot_name)/ee_gripper_link, mass 0.001
- added link $(arg robot_name)/left_finger_link, mass 0.034796; collision mesh filename=${mesh_directory}/gripper_finger.stl scale=0.001 0.001 0.001; visual mesh filename=${mesh_directory}/gripper_finger.stl scale=0.001 0.001 0.001
- added link $(arg robot_name)/right_finger_link, mass 0.034796; collision mesh filename=${mesh_directory}/gripper_finger.stl scale=0.001 0.001 0.001; visual mesh filename=${mesh_directory}/gripper_finger.stl scale=0.001 0.001 0.001
Joints:
- added joint ee_gripper: type fixed, parent $(arg robot_name)/fingers_link, child $(arg robot_name)/ee_gripper_link, origin xyz=0.0385 0 0 rpy=0 -${pi/2} 0, axis 1 0 0
- added joint left_finger: type prismatic, parent $(arg robot_name)/fingers_link, child $(arg robot_name)/left_finger_link, origin xyz=0 0 0 rpy=0 0 0, axis 0 1 0, limit lower=${finger_limit_lower} upper=${finger_limit_upper} effort=${finger_limit_effort} velocity=${finger_limit_vel}
- added joint right_finger: type prismatic, parent $(arg robot_name)/fingers_link, child $(arg robot_name)/right_finger_link, origin xyz=0 0 0 rpy=0 0 0, axis 0 1 0, limit lower=${-finger_limit_upper} upper=${-finger_limit_lower} effort=${finger_limit_effort} velocity=${finger_limit_vel}

Commit message: mafakka

File: code/src/husky_interbotix/urdf/interbotix_urdf_extras.urdf (robot description, URDF)
Before this commit: robot None, 2 links, 2 joints
Links:
- added link case
- added link case_link; visual box size=0.016 0.06 0.045
Joints:
- added joint case_joint: type fixed, parent case, child case_link, origin xyz=0.01 0 0.0 rpy=0 0 0

Commit message: jlkdjsg

File: code/src/husky_interbotix/urdf/interbotix_urdf_extras.urdf (robot description, URDF)
Before this commit: robot None, 4 links, 3 joints
Links:
- removed link case
- removed link case_link
Joints:
- removed joint case_joint

Commit message: heklo

File: code/src/husky_interbotix/urdf/interbotix_urdf_extras.urdf (robot description, URDF)
Before this commit: robot None, 2 links, 2 joints
Joints:
- joint camera_frame_joint: origin xyz=0.028 0 0.035 rpy=0 0 0 -> xyz=0.028 0.05 0.035 rpy=0 0 0

Commit message: hsjdh

File: code/src/husky_interbotix/urdf/interbotix_urdf_extras.urdf (robot description, URDF)
Before this commit: robot None, 2 links, 2 joints
Joints:
- joint camera_frame_joint: origin xyz=0.028 0.05 0.035 rpy=0 0 0 -> xyz=0.028 0.045 0.035 rpy=0 0 0

Commit message: bing bong

File: code/src/husky_interbotix/urdf/interbotix_urdf_extras.urdf (robot description, URDF)
Before this commit: robot None, 2 links, 2 joints
Joints:
- joint camera_frame_joint: origin xyz=0.028 0.045 0.035 rpy=0 0 0 -> xyz=0.028 0.045 0.025 rpy=0 0 0

Commit message: fak

File: code/src/husky_interbotix/urdf/interbotix_urdf_extras.urdf (robot description, URDF)
Before this commit: robot None, 2 links, 2 joints
Joints:
- joint camera_frame_joint: origin xyz=0.028 0.045 0.025 rpy=0 0 0 -> xyz=0.028 0 0.035 rpy=0 0 0
- joint realsense_joint: origin xyz=0.035 0 0.025 rpy=0 0 0 -> xyz=0.035 0.045 0.015 rpy=0 0 0

Commit message: small adjustment

File: code/src/husky_interbotix/urdf/interbotix_urdf_extras.urdf (robot description, URDF)
Before this commit: robot None, 2 links, 2 joints
Joints:
- joint realsense_joint: origin xyz=0.035 0.045 0.015 rpy=0 0 0 -> xyz=0.035 0.045 0.0125 rpy=0 0 0

Commit message: yes

File: code/src/husky_interbotix/urdf/interbotix_urdf_extras.urdf (robot description, URDF)
Before this commit: robot None, 2 links, 2 joints
Joints:
- joint realsense_joint: origin xyz=0.035 0.045 0.0125 rpy=0 0 0 -> xyz=0.035 0.045 0.0115 rpy=0 0 0

Commit message: hmm

File: code/src/husky_interbotix/urdf/interbotix_urdf_extras.urdf (robot description, URDF)
Before this commit: robot None, 2 links, 2 joints
Joints:
- joint realsense_joint: origin xyz=0.035 0.045 0.0115 rpy=0 0 0 -> xyz=0.035 0.045 0.0 rpy=0 0 0

Commit message: now

File: code/src/husky_interbotix/urdf/interbotix_urdf_extras.urdf (robot description, URDF)
Before this commit: robot None, 2 links, 2 joints
Joints:
- joint realsense_joint: origin xyz=0.035 0.045 0.0 rpy=0 0 0 -> xyz=0.035 0.045 0.013 rpy=0 0 0

Commit message: hei

File: code/src/husky_interbotix/urdf/interbotix_urdf_extras.urdf (robot description, URDF)
Before this commit: robot None, 2 links, 2 joints
Joints:
- joint realsense_joint: origin xyz=0.035 0.045 0.013 rpy=0 0 0 -> xyz=0.035 0.045 0.03 rpy=0 0 0

Commit message: hmm

File: code/src/husky_interbotix/urdf/interbotix_urdf_extras.urdf (robot description, URDF)
Before this commit: robot None, 2 links, 2 joints
Joints:
- joint realsense_joint: origin xyz=0.035 0.045 0.03 rpy=0 0 0 -> xyz=0.035 0.045 0.04 rpy=0 0 0

Commit message: jaman

File: code/src/husky_interbotix/urdf/interbotix_urdf_extras.urdf (robot description, URDF)
Before this commit: robot None, 2 links, 2 joints
Joints:
- joint realsense_joint: origin xyz=0.035 0.045 0.04 rpy=0 0 0 -> xyz=0.035 0.045 0.045 rpy=0 0 0

Commit message: haha

File: code/src/husky_interbotix/urdf/interbotix_urdf_extras.urdf (robot description, URDF)
Before this commit: robot None, 2 links, 2 joints
Joints:
- joint realsense_joint: origin xyz=0.035 0.045 0.045 rpy=0 0 0 -> xyz=0.035 0.045 0.035 rpy=0 0 0

Commit message: yes

File: code/src/husky_interbotix/urdf/interbotix_urdf_extras.urdf (robot description, URDF)
Before this commit: robot None, 2 links, 2 joints
Joints:
- joint realsense_joint: origin xyz=0.035 0.045 0.035 rpy=0 0 0 -> xyz=0.035 0.045 0.0325 rpy=0 0 0

Commit message: no

File: code/src/husky_interbotix/urdf/interbotix_urdf_extras.urdf (robot description, URDF)
Before this commit: robot None, 2 links, 2 joints
Joints:
- joint realsense_joint: origin xyz=0.035 0.045 0.0325 rpy=0 0 0 -> xyz=0.035 0.045 0.032 rpy=0 0 0

Commit message: hei

File: code/src/husky_interbotix/urdf/interbotix_urdf_extras.urdf (robot description, URDF)
Before this commit: robot None, 2 links, 2 joints
Joints:
- joint realsense_joint: origin xyz=0.035 0.045 0.032 rpy=0 0 0 -> xyz=0.015 0.045 0.032 rpy=0 0 0

Commit message: bang

File: code/src/husky_interbotix/urdf/interbotix_urdf_extras.urdf (robot description, URDF)
Before this commit: robot None, 2 links, 2 joints
Joints:
- joint realsense_joint: origin xyz=0.015 0.045 0.032 rpy=0 0 0 -> xyz=0.055 0.045 0.032 rpy=0 0 0

Commit message: fe

File: code/src/husky_interbotix/urdf/interbotix_urdf_extras.urdf (robot description, URDF)
Before this commit: robot None, 2 links, 2 joints
Joints:
- joint realsense_joint: origin xyz=0.055 0.045 0.032 rpy=0 0 0 -> xyz=0.05 0.045 0.032 rpy=0 0 0

Commit message: adjusted cam

File: code/src/husky_interbotix/urdf/interbotix_urdf_extras.urdf (robot description, URDF)
Before this commit: robot None, 2 links, 2 joints
Joints:
- joint realsense_joint: origin xyz=0.05 0.045 0.032 rpy=0 0 0 -> xyz=0.05+0.052348 0.045+0.053532 0.032 rpy=0 0 0

Commit message: math?

File: code/src/husky_interbotix/urdf/interbotix_urdf_extras.urdf (robot description, URDF)
Before this commit: robot None, 2 links, 2 joints
Joints:
- joint realsense_joint: origin xyz=0.05+0.052348 0.045+0.053532 0.032 rpy=0 0 0 -> xyz={0.05+0.052348} {0.045+0.053532} 0.032 rpy=0 0 0

Commit message: adjusted feil

File: code/src/husky_interbotix/urdf/interbotix_urdf_extras.urdf (robot description, URDF)
Before this commit: robot None, 2 links, 2 joints
Joints:
- joint realsense_joint: origin xyz={0.05+0.052348} {0.045+0.053532} 0.032 rpy=0 0 0 -> xyz=0.102348 0.0985 0.032 rpy=0 0 0

Commit message: too many decimals?

File: code/src/husky_interbotix/urdf/interbotix_urdf_extras.urdf (robot description, URDF)
Before this commit: robot None, 2 links, 2 joints
Joints:
- joint realsense_joint: origin xyz=0.102348 0.0985 0.032 rpy=0 0 0 -> xyz=0.10235 0.0985 0.032 rpy=0 0 0

Commit message: wahtta

File: code/src/husky_interbotix/urdf/interbotix_urdf_extras.urdf (robot description, URDF)
Before this commit: robot None, 2 links, 2 joints
Joints:
- joint realsense_joint: origin xyz=0.10235 0.0985 0.032 rpy=0 0 0 -> xyz=0.102348 0.0985 0.032 rpy=0 0 0

Commit message: test

File: code/src/husky_interbotix/urdf/interbotix_urdf_extras.urdf (robot description, URDF)
Before this commit: robot None, 2 links, 2 joints
Joints:
- joint realsense_joint: origin xyz=0.102348 0.0985 0.032 rpy=0 0 0 -> xyz=0.502348 0.5985 0.032 rpy=0 0 0

Commit message: dsjglksdfh

File: code/src/husky_interbotix/urdf/interbotix_urdf_extras.urdf (robot description, URDF)
Before this commit: robot None, 2 links, 2 joints
Joints:
- joint camera_frame_joint: origin xyz=0.028 0 0.035 rpy=0 0 0 -> xyz=0.080348 0 0.088532 rpy=0 0 0
- joint realsense_joint: origin xyz=0.502348 0.5985 0.032 rpy=0 0 0 -> xyz=0.05 0.5985 0.032 rpy=0 0 0

Commit message: fsdgsdgdfs

File: code/src/husky_interbotix/urdf/interbotix_urdf_extras.urdf (robot description, URDF)
Before this commit: robot None, 2 links, 2 joints
Joints:
- joint camera_frame_joint: origin xyz=0.080348 0 0.088532 rpy=0 0 0 -> xyz=0.028 0 0.035 rpy=0 0 0
- joint realsense_joint: origin xyz=0.05 0.5985 0.032 rpy=0 0 0 -> xyz=0.10235 0.0985 0.032 rpy=0 0 0

Commit message: joidfjugisd

File: code/src/husky_interbotix/urdf/interbotix_urdf_extras.urdf (robot description, URDF)
Before this commit: robot None, 2 links, 2 joints
Joints:
- joint realsense_joint: origin xyz=0.10235 0.0985 0.032 rpy=0 0 0 -> xyz=0.075856 0.071 0.032 rpy=0 0 0

Commit message: jk

File: code/src/husky_interbotix/urdf/interbotix_urdf_extras.urdf (robot description, URDF)
Before this commit: robot None, 2 links, 2 joints
Joints:
- joint realsense_joint: origin xyz=0.075856 0.071 0.032 rpy=0 0 0 -> xyz=0.05 0.045 0.032 rpy=0 0 0

Commit message: well

File: code/src/husky_interbotix/urdf/interbotix_urdf_extras.urdf (robot description, URDF)
Before this commit: robot None, 2 links, 2 joints
Joints:
- joint realsense_joint: origin xyz=0.05 0.045 0.032 rpy=0 0 0 -> xyz=0.05 0.045 0.006273 rpy=0 0 0

Commit message: trying

File: code/src/husky_interbotix/urdf/interbotix_urdf_extras.urdf (robot description, URDF)
Before this commit: robot None, 2 links, 2 joints
Joints:
- joint realsense_joint: origin xyz=0.05 0.045 0.006273 rpy=0 0 0 -> xyz=0.05 0.00 0.006273 rpy=0 0 0

Commit message: wellwellwell

File: code/src/husky_interbotix/urdf/interbotix_urdf_extras.urdf (robot description, URDF)
Before this commit: robot None, 2 links, 2 joints
Joints:
- joint realsense_joint: origin xyz=0.05 0.00 0.006273 rpy=0 0 0 -> xyz=0.05 0.001997 0.006273 rpy=0 0 0

Commit message: y adjust

File: code/src/husky_interbotix/urdf/interbotix_urdf_extras.urdf (robot description, URDF)
Before this commit: robot None, 2 links, 2 joints
Joints:
- joint realsense_joint: origin xyz=0.05 0.001997 0.006273 rpy=0 0 0 -> xyz=0.05 0.045 0.006273 rpy=0 0 0

Commit message: fakk

File: code/src/husky_interbotix/urdf/interbotix_urdf_extras.urdf (robot description, URDF)
Before this commit: robot None, 2 links, 2 joints
Joints:
- joint realsense_joint: origin xyz=0.05 0.045 0.006273 rpy=0 0 0 -> xyz=0.05 0.045 0.032 rpy=0 0 0
